File: hardware/ch32x035/uDap.kicad_pcb (KiCad board)
At the start: 2 copper layers, 27.2 x 11.8 mm, 18 parts, among them J1 USB_C_Receptacle_USB2.0_16P, J3 Conn_02x05_Odd_Even, SW3 SW_MEC_5E, U1 CH32X035F8U6, U2 RT9013

Commit message: Update uDap project files: change isolated pin label warning to error, add nRST label, and revise README with updated performance data
Connections:
- U1 pad 9: unconnected-(U1-PA7-Pad9) -> /nRST
Routing:
- net /nRST: track 0.00 -> 14.2 mm, vias 0 -> 1
