File: hardware/ch32x035/uDap.kicad_sch (KiCad schematic)
At the start: 18 parts, among them J1 USB_C_Receptacle_USB2.0_16P, J3 Conn_02x05_Odd_Even, SW3 SW_MEC_5E, U1 CH32X035F8U6, U2 RT9013

Commit message: Update uDap project files: change isolated pin label warning to error, add nRST label, and revise README with updated performance data
Connections:
- net nRST: now also U1.9 (PA7)
- no-connect marks 7 -> 6
Changed lines of the file:
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@@
-	)
-	(no_connect
-		(at 127 114.3)
 	)
 	(no_connect
@@
 		(effects
 			(font
+				(size 1.27 1.27)
+			)
+			(justify left bottom)
+		)
+	)
+	(label "nRST"
+		(at 127 114.3 0)
+		(effects
+			(font
